Commit message: fix

File: urdf/URDF.urdf (robot description, URDF)
Before this commit: robot URDF, 7 links, 6 joints
Joints:
- joint joint_1: type revolute -> continuous
- joint joint_2: limit lower=0 upper=0 effort=0 velocity=0 -> lower=-1.5 upper=1.5 effort=0 velocity=0
- joint joint_3: limit lower=0 upper=0 effort=0 velocity=0 -> lower=-3.1 upper=0.25 effort=0 velocity=0
- joint joint_4: type revolute -> continuous
- joint joint_5: limit lower=0 upper=0 effort=0 velocity=0 -> lower=-1.575 upper=1.575 effort=0 velocity=0
- joint joint_6: type revolute -> continuous
